Commit message: Addding leon to scenario

File: demos/models/obstacles/props/can/can.urdf (robot description, URDF)
Before this commit: robot can, 1 links, 0 joints
Links:
- link base: geometry collision cylinder length=0.11 radius=0.030; visual mesh filename=cokecan2.dae scale=0.0254 0.0254 0.0254
