Commit message: New lemon model functional

File: demos/models/obstacles/props/lemon/lemon.urdf (robot description, URDF)
Before this commit: robot lemon, 1 links, 0 joints
Links:
- link base: geometry collision mesh filename=lemon.dae scale=0.37 0.37 0.37; visual mesh filename=lemon.dae scale=0.37 0.37 0.37

Commit message: Resizing lemon to 0.3

File: demos/models/obstacles/props/lemon/lemon.urdf (robot description, URDF)
Before this commit: robot lemon, 1 links, 0 joints
Links:
- link base: geometry collision mesh filename=lemon.dae scale=0.3 0.3 0.3; visual mesh filename=lemon.dae scale=0.3 0.3 0.3
