Commit message: Adding v2 of the final problem including the multipick action

File: demos/models/obstacles/props/glass/glass.urdf (robot description, URDF)
Before this commit: robot glass, 1 links, 0 joints
Links:
- link base: geometry collision mesh filename=glass_v2.wrl scale=0.0035 0.0035 0.0035; visual mesh filename=glass_v2.wrl scale=0.0035 0.0035 0.0035
