Commit message: Adding second can for more difficult approach

File: demos/models/obstacles/restaurant/auxiliar_blocks/aux_prop.urdf (robot description, URDF)
Before this commit: robot aux_box_lemon, 1 links, 0 joints
Links:
- link base: geometry collision box size=0.001 0.001 0.075; visual box size=0.001 0.001 0.075
